Commit message: 更新
更新

File: src/my_robot_description/urdf/my_robot.urdf.xacro (robot description, xacro)
@@ -1,5 +1,17 @@
 <?xml version="1.0"?>
+<!--
+  Enhanced robot description with improved sensor configuration and parameters.
+  This file defines a differential drive mobile robot with:
+  - Parametrized physical dimensions
+  - Enhanced laser scanner configuration
+  - Improved Gazebo plugin integration
+  - Better material and visual properties
+-->
 <robot name="my_robot" xmlns:xacro="http://ros.org/xacro">
+  <!-- Include external parameter file -->
+  <xacro:property name="config_file" value="$(find my_robot_description)/config/robot_params.yaml" />
+  <!-- Mathematical constants -->
   <xacro:property name="M_PI" value="3.1415926535897931" />
+  <!-- Physical dimensions (can be overridden by config file) -->
   <xacro:property name="base_link_len" value="0.3" />
   <xacro:property name="base_link_width" value="0.2" />
@@ -8,4 +20,24 @@
   <xacro:property name="wheel_thickness" value="0.03" />
   <xacro:property name="wheel_separation" value="0.22" />
+  <xacro:property name="caster_radius" value="0.02" />
+  <!-- Sensor parameters -->
+  <xacro:property name="laser_size_x" value="0.05" />
+  <xacro:property name="laser_size_y" value="0.05" />
+  <xacro:property name="laser_size_z" value="0.03" />
+  <xacro:property name="laser_mass" value="0.1" />
+  <!-- Material definitions -->
+  <material name="blue">
+    <color rgba="0.2 0.4 0.8 1.0" />
+  </material>
+  <material name="black">
+    <color rgba="0.1 0.1 0.1 1.0" />
+  </material>
+  <material name="grey">
+    <color rgba="0.5 0.5 0.5 1.0" />
+  </material>
+  <material name="red">
+    <color rgba="0.8 0.2 0.2 1.0" />
+  </material>
+  <!-- Base link -->
   <link name="base_link">
     <visual>
@@ -13,7 +45,5 @@
         <box size="${base_link_len} ${base_link_width} ${base_link_height}" />
       </geometry>
-      <material name="blue">
-        <color rgba="0 0 1 1" />
-      </material>
+      <material name="blue" />
     </visual>
     <collision>
@@ -25,7 +55,9 @@
       <origin xyz="0 0 0" rpy="0 0 0" />
       <mass value="1.0" />
-      <inertia ixx="0.01" ixy="0.0" ixz="0.0" iyy="0.01" iyz="0.0" izz="0.01" />
-    </inertial>
-  </link>
+      <inertia ixx="0.0083" ixy="0.0" ixz="0.0"
+               iyy="0.0083" iyz="0.0" izz="0.0133" />
+    </inertial>
+  </link>
+  <!-- Left wheel -->
   <link name="left_wheel_link">
     <visual>
@@ -34,7 +66,5 @@
         <cylinder radius="${wheel_radius}" length="${wheel_thickness}" />
       </geometry>
-      <material name="black">
-        <color rgba="0 0 0 1" />
-      </material>
+      <material name="black" />
     </visual>
     <collision>
@@ -47,5 +77,6 @@
       <origin xyz="0 0 0" rpy="0 0 0" />
       <mass value="0.1" />
-      <inertia ixx="0.0001" ixy="0.0" ixz="0.0" iyy="0.0001" iyz="0.0" izz="0.0001" />
+      <inertia ixx="0.000125" ixy="0.0" ixz="0.0"
+               iyy="0.000125" iyz="0.0" izz="0.00025" />
     </inertial>
   </link>
@@ -56,4 +87,5 @@
     <axis xyz="0 1 0" />
   </joint>
+  <!-- Right wheel -->
   <link name="right_wheel_link">
     <visual>
@@ -73,5 +105,6 @@
       <origin xyz="0 0 0" rpy="0 0 0" />
       <mass value="0.1" />
-      <inertia ixx="0.0001" ixy="0.0" ixz="0.0" iyy="0.0001" iyz="0.0" izz="0.0001" />
+      <inertia ixx="0.000125" ixy="0.0" ixz="0.0"
+               iyy="0.000125" iyz="0.0" izz="0.00025" />
     </inertial>
   </link>
@@ -82,18 +115,17 @@
     <axis xyz="0 1 0" />
   </joint>
+  <!-- Caster wheel -->
   <link name="caster_link">
     <visual>
       <origin xyz="0 0 0" rpy="0 0 0" />
       <geometry>
-        <sphere radius="0.02" />
-      </geometry>
-      <material name="grey">
-        <color rgba="0.5 0.5 0.5 1" />
-      </material>
-    </visual>
-    <collision>
-      <origin xyz="0 0 0" rpy="0 0 0" />
-      <geometry>
-        <sphere radius="0.02" />
+        <sphere radius="${caster_radius}" />
+      </geometry>
+      <material name="grey" />
+    </visual>
+    <collision>
+      <origin xyz="0 0 0" rpy="0 0 0" />
+      <geometry>
+        <sphere radius="${caster_radius}" />
       </geometry>
     </collision>
@@ -101,5 +133,6 @@
       <origin xyz="0 0 0" rpy="0 0 0" />
       <mass value="0.01" />
-      <inertia ixx="0.00001" ixy="0.0" ixz="0.0" iyy="0.00001" iyz="0.0" izz="0.00001" />
+      <inertia ixx="0.0000016" ixy="0.0" ixz="0.0"
+               iyy="0.0000016" iyz="0.0" izz="0.0000016" />
     </inertial>
   </link>
@@ -107,6 +140,34 @@
     <parent link="base_link" />
     <child link="caster_link" />
-    <origin xyz="-0.1 0 ${-(base_link_height/2 - 0.02)}" rpy="0 0 0" />
-  </joint>
+    <origin xyz="-${base_link_len/2 - caster_radius} 0 ${-(base_link_height/2 + caster_radius)}" rpy="0 0 0" />
+  </joint>
+  <!-- Laser scanner link -->
+  <link name="laser_link">
+    <visual>
+      <origin xyz="0 0 0" rpy="0 0 0" />
+      <geometry>
+        <box size="${laser_size_x} ${laser_size_y} ${laser_size_z}" />
+      </geometry>
+      <material name="red" />
+    </visual>
+    <collision>
+      <origin xyz="0 0 0" rpy="0 0 0" />
+      <geometry>
+        <box size="${laser_size_x} ${laser_size_y} ${laser_size_z}" />
+      </geometry>
+    </collision>
+    <inertial>
+      <origin xyz="0 0 0" rpy="0 0 0" />
+      <mass value="${laser_mass}" />
+      <inertia ixx="0.0000833" ixy="0.0" ixz="0.0"
+               iyy="0.0000833" iyz="0.0" izz="0.0000833" />
+    </inertial>
+  </link>
+  <joint name="laser_joint" type="fixed">
+    <parent link="base_link" />
+    <child link="laser_link" />
+    <origin xyz="${base_link_len/2 - laser_size_x/2} 0 ${base_link_height/2 + laser_size_z/2}" rpy="0 0 0" />
+  </joint>
+  <!-- Gazebo differential drive plugin -->
   <gazebo>
     <plugin name="differential_drive_controller" filename="libgazebo_ros_diff_drive.so">
@@ -119,15 +180,20 @@
       <right_joint>right_wheel_joint</right_joint>
       <wheel_separation>${wheel_separation}</wheel_separation>
-      <wheel_radius>${wheel_radius}</wheel_radius>
-      <publish_tf>true</publish_tf>
+      <wheel_diameter>${2 * wheel_radius}</wheel_diameter>
+      <max_wheel_torque>20</max_wheel_torque>
+      <max_wheel_acceleration>1.0</max_wheel_acceleration>
       <publish_odom>true</publish_odom>
+      <publish_odom_tf>true</publish_odom_tf>
       <publish_wheel_tf>false</publish_wheel_tf>
       <odometry_frame>odom</odometry_frame>
       <robot_base_frame>base_link</robot_base_frame>
+      <update_rate>50.0</update_rate>
     </plugin>
   </gazebo>
-  <gazebo reference="base_link">
-    <sensor type="ray" name="my_robot_laser_sensor">
-      <pose>0.1 0 ${base_link_height/2 + 0.02} 0 0 0</pose> <visualize>true</visualize>
+  <!-- Gazebo laser scanner plugin -->
+  <gazebo reference="laser_link">
+    <sensor type="ray" name="laser_scanner">
+      <pose>0 0 0 0 0 0</pose>
+      <visualize>true</visualize>
       <update_rate>10</update_rate>
       <ray>
@@ -145,10 +211,53 @@
           <resolution>0.01</resolution>
         </range>
+        <noise>
+          <type>gaussian</type>
+          <mean>0.0</mean>
+          <stddev>0.01</stddev>
+        </noise>
       </ray>
-      <plugin name="laser_controller" filename="libgazebo_ros_laser.so">
-        <topicName>scan</topicName>
-        <frameName>laser_link</frameName>
+      <plugin name="gazebo_ros_laser" filename="libgazebo_ros_ray_sensor.so">
+        <ros>
+          <namespace>/</namespace>
+          <argument>~/out:=scan</argument>
+        </ros>
+        <output_type>sensor_msgs/LaserScan</output_type>
+        <frame_name>laser_link</frame_name>
       </plugin>
     </sensor>
   </gazebo>
+  <!-- Gazebo material properties -->
+  <gazebo reference="base_link">
+    <material>Gazebo/Blue</material>
+  </gazebo>
+  <gazebo reference="left_wheel_link">
+    <material>Gazebo/Black</material>
+    <mu1>1.0</mu1>
+    <mu2>1.0</mu2>
+    <kp>500000.0</kp>
+    <kd>10.0</kd>
+    <minDepth>0.001</minDepth>
+    <maxVel>0.1</maxVel>
+  </gazebo>
+  <gazebo reference="right_wheel_link">
+    <material>Gazebo/Black</material>
+    <mu1>1.0</mu1>
+    <mu2>1.0</mu2>
+    <kp>500000.0</kp>
+    <kd>10.0</kd>
+    <minDepth>0.001</minDepth>
+    <maxVel>0.1</maxVel>
+  </gazebo>
+  <gazebo reference="caster_link">
+    <material>Gazebo/Grey</material>
+    <mu1>0.1</mu1>
+    <mu2>0.1</mu2>
+    <kp>500000.0</kp>
+    <kd>10.0</kd>
+    <minDepth>0.001</minDepth>
+    <maxVel>0.1</maxVel>
+  </gazebo>
+  <gazebo reference="laser_link">
+    <material>Gazebo/Red</material>
+  </gazebo>
 </robot>
