Commit message: text

File: src/my_robot_description/urdf/model.urdf (robot description, URDF)
Before this commit: robot my_robot, 5 links, 4 joints
Links:
- added link camera_link, mass 0.05; collision box size=0.04 0.04 0.04; visual box size=0.04 0.04 0.04
Joints:
- added joint camera_joint: type fixed, parent base_link, child camera_link, origin xyz=0.2 0 0.15000000000000002 rpy=0 0 0

File: src/my_robot_description/urdf/my_robot.urdf.xacro (robot description, xacro)
@@ -169,4 +169,31 @@
     <origin xyz="${base_link_len/2 - laser_size_x/2} 0 ${base_link_height/2 + laser_size_z/2}" rpy="0 0 0" />
   </joint>
+  <!-- Camera link -->
+  <link name="camera_link">
+    <visual>
+      <origin xyz="0 0 0" rpy="0 0 0" />
+      <geometry>
+        <box size="0.04 0.04 0.04" />
+      </geometry>
+      <material name="grey" />
+    </visual>
+    <collision>
+      <origin xyz="0 0 0" rpy="0 0 0" />
+      <geometry>
+        <box size="0.04 0.04 0.04" />
+      </geometry>
+    </collision>
+    <inertial>
+      <origin xyz="0 0 0" rpy="0 0 0" />
+      <mass value="0.05" />
+      <inertia ixx="0.00001" ixy="0.0" ixz="0.0"
+               iyy="0.00001" iyz="0.0" izz="0.00001" />
+    </inertial>
+  </link>
+  <joint name="camera_joint" type="fixed">
+    <parent link="base_link" />
+    <child link="camera_link" />
+    <origin xyz="${base_link_len/2 + 0.05} 0 ${base_link_height/2 + 0.1}" rpy="0 0 0" />
+  </joint>
   <!-- Gazebo differential drive plugin -->
   <gazebo>
@@ -261,3 +288,31 @@
     <material>Gazebo/Red</material>
   </gazebo>
+  <!-- Gazebo camera sensor plugin -->
+  <gazebo reference="camera_link">
+    <sensor type="camera" name="camera_sensor">
+      <pose>0 0 0 0 0 0</pose>
+      <visualize>true</visualize>
+      <update_rate>15</update_rate>
+      <camera>
+        <horizontal_fov>1.047</horizontal_fov>
+        <image>
+          <width>640</width>
+          <height>480</height>
+          <format>R8G8B8</format>
+        </image>
+        <clip>
+          <near>0.05</near>
+          <far>10.0</far>
+        </clip>
+      </camera>
+      <plugin name="gazebo_ros_camera" filename="libgazebo_ros_camera.so">
+        <ros>
+          <namespace>/</namespace>
+          <remapping>image_raw:=/camera/image_raw</remapping>
+        </ros>
+        <camera_name>camera</camera_name>
+        <frame_name>camera_link</frame_name>
+      </plugin>
+    </sensor>
+  </gazebo>
 </robot>

Commit message: test1

File: src/my_robot_description/urdf/model.urdf (robot description, URDF)
Before this commit: robot my_robot, 6 links, 5 joints
Links:
- added link camera_optical_link
- link camera_link: mass 0.05 -> 0.072; geometry collision box size=0.09 0.025 0.025; visual box size=0.09 0.025 0.025
Joints:
- added joint camera_optical_joint: type fixed, parent camera_link, child camera_optical_link, origin xyz=0 0 0 rpy=-1.5707963267948966 0 -1.5707963267948966
- joint caster_joint: origin xyz=-0.13 0 -0.07 rpy=0 0 0 -> xyz=-0.13 0 -0.030000000000000002 rpy=0 0 0

File: src/my_robot_description/urdf/my_robot.urdf.xacro (robot description, xacro)
@@ -53,5 +53,5 @@
     </collision>
     <inertial>
-      <origin xyz="0 0 0" rpy="0 0 0" />
+      <origin xyz="-0.02 0 0" rpy="0 0 0" />
       <mass value="1.0" />
       <inertia ixx="0.0083" ixy="0.0" ixz="0.0"
@@ -140,5 +140,5 @@
     <parent link="base_link" />
     <child link="caster_link" />
-    <origin xyz="-${base_link_len/2 - caster_radius} 0 ${-(base_link_height/2 + caster_radius)}" rpy="0 0 0" />
+    <origin xyz="-${base_link_len/2 - caster_radius} 0 ${-(wheel_radius - caster_radius)}" rpy="0 0 0" />
   </joint>
   <!-- Laser scanner link -->
@@ -169,10 +169,10 @@
     <origin xyz="${base_link_len/2 - laser_size_x/2} 0 ${base_link_height/2 + laser_size_z/2}" rpy="0 0 0" />
   </joint>
-  <!-- Camera link -->
+  <!-- RGB-D Camera link (Intel RealSense style) -->
   <link name="camera_link">
     <visual>
       <origin xyz="0 0 0" rpy="0 0 0" />
       <geometry>
-        <box size="0.04 0.04 0.04" />
+        <box size="0.09 0.025 0.025" />
       </geometry>
       <material name="grey" />
@@ -181,10 +181,10 @@
       <origin xyz="0 0 0" rpy="0 0 0" />
       <geometry>
-        <box size="0.04 0.04 0.04" />
-      </geometry>
-    </collision>
-    <inertial>
-      <origin xyz="0 0 0" rpy="0 0 0" />
-      <mass value="0.05" />
+        <box size="0.09 0.025 0.025" />
+      </geometry>
+    </collision>
+    <inertial>
+      <origin xyz="0 0 0" rpy="0 0 0" />
+      <mass value="0.072" />
       <inertia ixx="0.00001" ixy="0.0" ixz="0.0"
                iyy="0.00001" iyz="0.0" izz="0.00001" />
@@ -195,4 +195,11 @@
     <child link="camera_link" />
     <origin xyz="${base_link_len/2 + 0.05} 0 ${base_link_height/2 + 0.1}" rpy="0 0 0" />
+  </joint>
+  <!-- Camera optical frame -->
+  <link name="camera_optical_link" />
+  <joint name="camera_optical_joint" type="fixed">
+    <parent link="camera_link" />
+    <child link="camera_optical_link" />
+    <origin xyz="0 0 0" rpy="-${M_PI/2} 0 -${M_PI/2}" />
   </joint>
   <!-- Gazebo differential drive plugin -->
@@ -288,10 +295,10 @@
     <material>Gazebo/Red</material>
   </gazebo>
-  <!-- Gazebo camera sensor plugin -->
+  <!-- Gazebo RGB-D camera sensor plugin -->
   <gazebo reference="camera_link">
-    <sensor type="camera" name="camera_sensor">
+    <sensor type="depth" name="camera_sensor">
       <pose>0 0 0 0 0 0</pose>
       <visualize>true</visualize>
-      <update_rate>15</update_rate>
+      <update_rate>30</update_rate>
       <camera>
         <horizontal_fov>1.047</horizontal_fov>
@@ -303,6 +310,11 @@
         <clip>
           <near>0.05</near>
-          <far>10.0</far>
+          <far>8.0</far>
         </clip>
+        <noise>
+          <type>gaussian</type>
+          <mean>0.0</mean>
+          <stddev>0.007</stddev>
+        </noise>
       </camera>
       <plugin name="gazebo_ros_camera" filename="libgazebo_ros_camera.so">
@@ -310,7 +322,12 @@
           <namespace>/</namespace>
           <remapping>image_raw:=/camera/image_raw</remapping>
+          <remapping>image_depth:=/camera/depth/image_raw</remapping>
+          <remapping>camera_info:=/camera/camera_info</remapping>
+          <remapping>depth/camera_info:=/camera/depth/camera_info</remapping>
+          <remapping>points:=/camera/points</remapping>
         </ros>
         <camera_name>camera</camera_name>
-        <frame_name>camera_link</frame_name>
+        <frame_name>camera_optical_link</frame_name>
+        <hack_baseline>0.07</hack_baseline>
       </plugin>
     </sensor>
